File: pcb/stm32l476rg_barebones/stm32l476rg.sch (KiCad schematic (older format))
At the start: 3 parts

Commit message: Schematic layout done
Parts:
- added C1: 4u7, symbol Device:C_Small
- added C10, C11, C12: 10u, symbol Device:C_Small
- added C13, C14: 12p, symbol Device:C_Small
- added C2, C3, C4, C5, C6: 100n, symbol Device:C_Small
- added C7, C9: 10n, symbol Device:C_Small
- added C8: 1u, symbol Device:C_Small
- added D1, D2: B5819W, symbol Device:D_Schottky
- added D3: YELLOW, symbol Device:LED_Small
- added D4: GREEN, symbol Device:LED_Small
- added F1: Polyfuse_Small, symbol Device:Polyfuse_Small
- added FB1: 600 @ 600MHz, symbol Device:Ferrite_Bead_Small
- added J1, J2: Conn_01x04, symbol Connector_Generic:Conn_01x04
- added J3: SWD_Connector, symbol Connector_Generic:Conn_02x05_Odd_Even
- added J4: Conn_01x06, symbol Connector_Generic:Conn_01x06
- added J5: USB_B_Micro, symbol Connector:USB_B_Micro
- added J6: Screw_Terminal_01x02, symbol Connector:Screw_Terminal_01x02
- added L1: 39n, symbol Device:L_Small
- added L2: 10u, symbol Device:L_Small
- added Q1: AO3401A, Package_TO_SOT_SMD:SOT-23, symbol Transistor_FET:AO3401A
- added R1, R2: 2K2, symbol Device:R_Small
- added R10: 1K, symbol Device:R_Small
- added R11: 1K5, symbol Device:R_Small
- added R4: 100K, symbol Device:R_Small
- added R5: 68K, symbol Device:R_Small
- added R6: 47K, symbol Device:R_Small
- added R7: 15K, symbol Device:R_Small
- added R8: 270, symbol Device:R_Small
- added R9: 47, symbol Device:R_Small
- added U1: USBLC6-2SC6, Package_TO_SOT_SMD:SOT-23-6, symbol Power_Protection:USBLC6-2SC6
- added U2: MP2359DJ-LF-Z, symbol STM32_Startup:MP2359DJ-LF-Z
- added Y1: HSE_4MHz, symbol Device:Crystal_GND24_Small
- gave numbers to parts that had none: 3
Connections:
- net GNDA is gone; now on net GND: U3.12 (VSSA)
- net +3.3VA: now also C8.1, C9.1, L1.2
- net +3V3: now also C1.1, C11.2, C12.2, C2.1, C3.1, C4.1, C5.1, C6.1, D3.2 (A), J1.1 (Pin_1), J2.1 (Pin_1), J3.1 (Pin_1), J4.1 (Pin_1), L1.1, L2.2, R1.1, R2.1, R6.1
- net GND: now also C1.2, C10.1, C11.1, C12.1, C13.1, C14.1, C2.2, C3.2, C4.2, C5.2, C6.2, C8.2, C9.2, D2.2 (A), J1.4 (Pin_4), J2.4 (Pin_4), J3.3 (Pin_3), J3.5 (Pin_5), J3.9 (Pin_9), J4.6 (Pin_6), J5.5 (GND), J6.2 (Pin_2), Q1.1 (G), R10.2, R11.2, R5.2, R8.2, U1.2 (GND), U2.2 (GND), Y1.2, Y1.4
- net HSE_IN: now also C13.2, Y1.1
- net HSE_OUT: now also R9.1
- net I2C1_SCL: now also J1.2 (Pin_2), R1.2
- net I2C1_SDA: now also J1.3 (Pin_3), R2.2
- net NRST: now also J3.10 (Pin_10)
- net SWCLK: now also J3.4 (Pin_4)
- net SWIDO: now also J3.2 (Pin_2)
- net SWO: now also J3.6 (Pin_6)
- net UART3_RX: now also J2.3 (Pin_3)
- net UART3_TX: now also J2.2 (Pin_2)
- net USB_D+: now also U1.4 (I/O2)
- net USB_D-: now also U1.6 (I/O1)
- net SPI1_CS1: now reaches U3.20 (PA4)
- net SPI1_CS1: now also J4.2 (Pin_2)
- net SPI1_SCK: now reaches U3.21 (PA5)
- net SPI1_SCK: now also J4.3 (Pin_3)
- net SPI1_MISO: now reaches U3.22 (PA6)
- net SPI1_MISO: now also J4.4 (Pin_4)
- net SPI1_MOSI: now reaches U3.23 (PA7)
- net SPI1_MOSI: now also J4.5 (Pin_5)
- net LED_STATUS: now reaches U3.39 (PC8)
- net LED_STATUS: now also D4.2 (A)
- new net: F1.1, Q1.3 (D)
- new net: D1.1 (K), FB1.2, Q1.2 (S)
- new net: C14.2, R9.2, Y1.3
- new net: R7.2, R8.1
- new net: D4.1 (K), R11.1
- new net: D3.1 (K), R10.1
- new net +5V: D1.2 (A), J5.1 (VBUS), U1.5 (VBUS)
- new net +9V: F1.2, J6.1 (Pin_1)
- new net BUCK_BST: C7.2, U2.1 (BST)
- new net BUCK_EN: R4.2, R5.1, U2.4 (EN)
- new net BUCK_FB: R6.2, R7.1, U2.3 (FB)
- new net BUCK_IN: C10.2, FB1.1, R4.1, U2.5 (IN)
- new net BUCK_SW: C7.1, D2.1 (K), L2.1, U2.6 (SW)
- new net USB_CONN_D+: J5.3 (D+), U1.3 (I/O2)
- new net USB_CONN_D-: J5.2 (D-), U1.1 (I/O1)
- no-connect marks 0 -> 39
Other:
- note added: "CLoad = 2 * [CLoadCrystal - Cstray]"
- note added: "Can add protective resistors to limit short circuit current on the peripheral lines"
- note added: "Can add to Pin_10 a decouple capacitor \nto avoid parasitic debouncing of reset\n"
- note added: "Connect Pin_8 if using JTAG\n"
- note added: "Debugger"
- note added: "I2C"
- note added: "Power Circuitry\n"
- note added: "SPI"
- note added: "STM32 MCU Run"
- note added: "UART"
- note added: "USB"
- moved on the sheet: R3, SW1, U3
