File: pcb/stm32l476rg_barebones/stm32l476rg.sch (KiCad schematic (older format))
At the start: 49 parts, among them J1 Conn_01x04_UART, J2 Conn_01x04_I2C, J3 Conn_01x06_SPI, J4 SWD_Connector, J5 USB_B_Micro, J6 Screw_Terminal_01x02, Q1 AO3401A, SW1 SW_SPDT, U1 USBLC6-2SC6, U2 MP2359DJ-LF-Z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

Commit message: Traced barebones
Connections:
- net +9V: now also Q1.3 (D); no longer F1.2
- net SPI1_CS1: now also U3.24 (PC4); no longer U3.20 (PA4)
- net at F1.1: now also FB1.2; no longer Q1.3 (D)
- net at D1.1 (K), Q1.2 (S): now also F1.2; no longer FB1.2
Other:
- moved on the sheet: C10, D1, F1, FB1, Q1
Changed lines of the file:
@@
 NoConn ~ 2800 6100
 NoConn ~ 2800 6000
-NoConn ~ 2800 5900
 NoConn ~ 2800 5800
 NoConn ~ 2800 5700
@@
 Text GLabel 4250 2000 0    50   Input ~ 0
 I2C1_SCL
-$Comp
-L Device:R_Small R2
-U 1 1 60F0FC72
-P 4750 1800
-F 0 "R2" H 4809 1846 50  0000 L CNN
-F 1 "2K2" H 4809 1755 50  0000 L CNN
-F 2 "Resistor_SMD:R_0603_1608Metric" H 4750 1800 50  0001 C CNN
-F 3 "~" H 4750 1800 50  0001 C CNN
-	1    4750 1800
-	1    0    0    -1
-$EndComp
-$Comp
-L Device:R_Small R1
-U 1 1 60F0B415
-P 4450 1800
-F 0 "R1" H 4509 1846 50  0000 L CNN
-F 1 "2K2" H 4509 1755 50  0000 L CNN
-F 2 "Resistor_SMD:R_0603_1608Metric" H 4450 1800 50  0001 C CNN
-F 3 "~" H 4450 1800 50  0001 C CNN
-	1    4450 1800
-	1    0    0    -1
-$EndComp
-Wire Wire Line
-	4250 2000 4450 2000
-Wire Wire Line
-	4450 2000 4450 1900
-Wire Wire Line
-	4250 2100 4750 2100
-Wire Wire Line
-	4750 2100 4750 1900
-$Comp
-L power:+3V3 #PWR012
-U 1 1 60F10299
-P 4450 1700
-F 0 "#PWR012" H 4450 1550 50  0001 C CNN
-F 1 "+3V3" H 4465 1873 50  0000 C CNN
-F 2 "" H 4450 1700 50  0001 C CNN
-F 3 "" H 4450 1700 50  0001 C CNN
-	1    4450 1700
-	1    0    0    -1
-$EndComp
-$Comp
-L power:+3V3 #PWR013
-U 1 1 60F11531
-P 4750 1700
-F 0 "#PWR013" H 4750 1550 50  0001 C CNN
-F 1 "+3V3" H 4765 1873 50  0000 C CNN
-F 2 "" H 4750 1700 50  0001 C CNN
-F 3 "" H 4750 1700 50  0001 C CNN
-	1    4750 1700
-	1    0    0    -1
-$EndComp
 Text GLabel 4250 1000 0    50   Input ~ 0
 I2C1_SCL
@@
 Text GLabel 4200 4300 2    50   Input ~ 0
 SPI1_SCK
-Text GLabel 4200 4200 2    50   Input ~ 0
+Text GLabel 2800 5900 0    50   Input ~ 0
 SPI1_CS1
 Text GLabel 5650 1300 0    50   Input ~ 0
@@
 Wire Wire Line
 	2750 2700 2350 2700
-Connection ~ 5650 3150
+Connection ~ 5800 3100
 $Comp
 L power:PWR_FLAG #FLG02
 U 1 1 610A764C
-P 5650 3150
-F 0 "#FLG02" H 5650 3225 50  0001 C CNN
-F 1 "PWR_FLAG" H 5650 3323 50  0000 C CNN
-F 2 "" H 5650 3150 50  0001 C CNN
-F 3 "~" H 5650 3150 50  0001 C CNN
-	1    5650 3150
+P 5800 3100
+F 0 "#FLG02" H 5800 3175 50  0001 C CNN
+F 1 "PWR_FLAG" H 5800 3273 50  0000 C CNN
+F 2 "" H 5800 3100 50  0001 C CNN
+F 3 "~" H 5800 3100 50  0001 C CNN
+	1    5800 3100
 	-1   0    0    1
 $EndComp
@@
 L power:+5V #PWR016
 U 1 1 60FC8FC9
-P 6900 2750
-F 0 "#PWR016" H 6900 2600 50  0001 C CNN
-F 1 "+5V" H 6915 2923 50  0000 C CNN
-F 2 "" H 6900 2750 50  0001 C CNN
-F 3 "" H 6900 2750 50  0001 C CNN
-	1    6900 2750
-	1    0    0    -1
-$EndComp
-Wire Wire Line
-	6900 3150 7550 3150
-Connection ~ 6900 3150
-Wire Wire Line
-	6900 3050 6900 3150
-Wire Wire Line
-	6750 3150 6900 3150
-$Comp
-L Device:D_Schottky D1
-U 1 1 60FAC885
-P 6900 2900
-F 0 "D1" V 6946 2820 50  0000 R CNN
-F 1 "B5819W" V 6855 2820 50  0000 R CNN
-F 2 "Diode_SMD:D_SOD-123" H 6900 2900 50  0001 C CNN
-F 3 "~" H 6900 2900 50  0001 C CNN
-	1    6900 2900
-	0    -1   -1   0
-$EndComp
+P 6600 2700
+F 0 "#PWR016" H 6600 2550 50  0001 C CNN
+F 1 "+5V" H 6615 2873 50  0000 C CNN
+F 2 "" H 6600 2700 50  0001 C CNN
+F 3 "" H 6600 2700 50  0001 C CNN
+	1    6600 2700
+	1    0    0    -1
+$EndComp
+Wire Wire Line
+	6600 3000 6600 3100
+Wire Wire Line
+	6450 3100 6600 3100
 $Comp
 L Connector:Screw_Terminal_01x02 J6
@@
 L power:+9V #PWR020
 U 1 1 60D39E06
-P 5650 3050
-F 0 "#PWR020" H 5650 2900 50  0001 C CNN
-F 1 "+9V" H 5665 3223 50  0000 C CNN
-F 2 "" H 5650 3050 50  0001 C CNN
-F 3 "" H 5650 3050 50  0001 C CNN
-	1    5650 3050
+P 5800 3000
+F 0 "#PWR020" H 5800 2850 50  0001 C CNN
+F 1 "+9V" H 5815 3173 50  0000 C CNN
+F 2 "" H 5800 3000 50  0001 C CNN
+F 3 "" H 5800 3000 50  0001 C CNN
+	1    5800 3000
 	1    0    0    -1
 $EndComp
@@
 L Device:Polyfuse_Small F1
 U 1 1 60D3A65B
-P 6000 3150
-F 0 "F1" V 5795 3150 50  0000 C CNN
-F 1 "250mA" V 5886 3150 50  0000 C CNN
-F 2 "Fuse:Fuse_1206_3216Metric" H 6050 2950 50  0001 L CNN
-F 3 "~" H 6000 3150 50  0001 C CNN
-	1    6000 3150
+P 6900 3100
+F 0 "F1" V 6800 3100 50  0000 C CNN
+F 1 "250mA" V 7000 3100 50  0000 C CNN
+F 2 "Fuse:Fuse_1206_3216Metric" H 6950 2900 50  0001 L CNN
+F 3 "~" H 6900 3100 50  0001 C CNN
+	1    6900 3100
 	0    1    1    0
 $EndComp
 Wire Wire Line
-	5650 3050 5650 3150
-Wire Wire Line
-	5650 3150 5900 3150
+	5800 3000 5800 3100
+Wire Wire Line
+	5800 3100 6050 3100
 $Comp
 L Transistor_FET:AO3401A Q1
 U 1 1 60D3E799
-P 6550 3250
-F 0 "Q1" V 6892 3250 50  0000 C CNN
-F 1 "AO3401A" V 6801 3250 50  0000 C CNN
-F 2 "Package_TO_SOT_SMD:SOT-23" H 6750 3175 50  0001 L CIN
-F 3 "http://www.aosmd.com/pdfs/datasheet/AO3401A.pdf" H 6550 3250 50  0001 L CNN
-	1    6550 3250
-	0    -1   -1   0
-$EndComp
-Wire Wire Line
-	6100 3150 6350 3150
+P 6250 3200
+F 0 "Q1" V 6592 3200 50  0000 C CNN
+F 1 "AO3401A" V 6501 3200 50  0000 C CNN
+F 2 "Package_TO_SOT_SMD:SOT-23" H 6450 3125 50  0001 L CIN
+F 3 "http://www.aosmd.com/pdfs/datasheet/AO3401A.pdf" H 6250 3200 50  0001 L CNN
+	1    6250 3200
+	0    -1   -1   0
+$EndComp
 $Comp
 L power:GND #PWR023
 U 1 1 60D44D8F
-P 6550 3450
-F 0 "#PWR023" H 6550 3200 50  0001 C CNN
-F 1 "GND" H 6555 3277 50  0000 C CNN
-F 2 "" H 6550 3450 50  0001 C CNN
-F 3 "" H 6550 3450 50  0001 C CNN
-	1    6550 3450
+P 6250 3400
+F 0 "#PWR023" H 6250 3150 50  0001 C CNN
+F 1 "GND" H 6255 3227 50  0000 C CNN
+F 2 "" H 6250 3400 50  0001 C CNN
+F 3 "" H 6250 3400 50  0001 C CNN
+	1    6250 3400
 	1    0    0    -1
 $EndComp
@@
 L Device:Ferrite_Bead_Small FB1
 U 1 1 60D46616
-P 7650 3150
-F 0 "FB1" V 7413 3150 50  0000 C CNN
-F 1 "600 @ 600MHz" V 7504 3150 50  0000 C CNN
-F 2 "Inductor_SMD:L_0805_2012Metric" V 7580 3150 50  0001 C CNN
-F 3 "~" H 7650 3150 50  0001 C CNN
-	1    7650 3150
+P 7350 3100
+F 0 "FB1" V 7113 3100 50  0000 C CNN
+F 1 "600 @ 600MHz" V 7204 3100 50  0000 C CNN
+F 2 "Inductor_SMD:L_0805_2012Metric" V 7280 3100 50  0001 C CNN
+F 3 "~" H 7350 3100 50  0001 C CNN
+	1    7350 3100
 	0    1    1    0
 $EndComp
@@
 L power:GND #PWR024
 U 1 1 60D4D250
-P 8000 3450
-F 0 "#PWR024" H 8000 3200 50  0001 C CNN
-F 1 "GND" H 8005 3277 50  0000 C CNN
-F 2 "" H 8000 3450 50  0001 C CNN
-F 3 "" H 8000 3450 50  0001 C CNN
-	1    8000 3450
-	1    0    0    -1
-$EndComp
-Text GLabel 8300 3150 2    50   Input ~ 0
+P 7700 3400
+F 0 "#PWR024" H 7700 3150 50  0001 C CNN
+F 1 "GND" H 7705 3227 50  0000 C CNN
+F 2 "" H 7700 3400 50  0001 C CNN
+F 3 "" H 7700 3400 50  0001 C CNN
+	1    7700 3400
+	1    0    0    -1
+$EndComp
+Text GLabel 8000 3100 2    50   Input ~ 0
 BUCK_IN
 Wire Wire Line
-	7750 3150 8000 3150
-Wire Wire Line
-	8000 3150 8000 3250
-Connection ~ 8000 3150
-Wire Wire Line
-	8000 3150 8300 3150
+	7450 3100 7700 3100
+Wire Wire Line
+	7700 3100 7700 3200
+Connection ~ 7700 3100
+Wire Wire Line
+	7700 3100 8000 3100
 Wire Wire Line
 	6800 4400 6800 4500
@@
 L Device:C_Small C10
 U 1 1 60D4B199
-P 8000 3350
-F 0 "C10" H 7908 3304 50  0000 R CNN
-F 1 "10u" H 7908 3395 50  0000 R CNN
-F 2 "Capacitor_SMD:C_1206_3216Metric" H 8000 3350 50  0001 C CNN
-F 3 "~" H 8000 3350 50  0001 C CNN
-	1    8000 3350
+P 7700 3300
+F 0 "C10" H 7608 3254 50  0000 R CNN
+F 1 "10u" H 7608 3345 50  0000 R CNN
+F 2 "Capacitor_SMD:C_1206_3216Metric" H 7700 3300 50  0001 C CNN
+F 3 "~" H 7700 3300 50  0001 C CNN
+	1    7700 3300
 	-1   0    0    1
 $EndComp
@@
 	1    0    0    -1
 $EndComp
+Wire Wire Line
+	4250 2100 4750 2100
+Wire Wire Line
+	4250 2000 4450 2000
+$Comp
+L power:+3V3 #PWR013
+U 1 1 60F11531
+P 4750 1700
+F 0 "#PWR013" H 4750 1550 50  0001 C CNN
+F 1 "+3V3" H 4765 1873 50  0000 C CNN
+F 2 "" H 4750 1700 50  0001 C CNN
+F 3 "" H 4750 1700 50  0001 C CNN
+	1    4750 1700
+	1    0    0    -1
+$EndComp
+$Comp
+L power:+3V3 #PWR012
+U 1 1 60F10299
+P 4450 1700
+F 0 "#PWR012" H 4450 1550 50  0001 C CNN
+F 1 "+3V3" H 4465 1873 50  0000 C CNN
+F 2 "" H 4450 1700 50  0001 C CNN
+F 3 "" H 4450 1700 50  0001 C CNN
+	1    4450 1700
+	1    0    0    -1
+$EndComp
+Wire Wire Line
+	4750 2100 4750 1900
+Wire Wire Line
+	4450 2000 4450 1900
+$Comp
+L Device:R_Small R1
+U 1 1 60F0B415
+P 4450 1800
+F 0 "R1" H 4509 1846 50  0000 L CNN
+F 1 "2K2" H 4509 1755 50  0000 L CNN
+F 2 "Resistor_SMD:R_0603_1608Metric" H 4450 1800 50  0001 C CNN
+F 3 "~" H 4450 1800 50  0001 C CNN
+	1    4450 1800
+	1    0    0    -1
+$EndComp
+$Comp
+L Device:R_Small R2
+U 1 1 60F0FC72
+P 4750 1800
+F 0 "R2" H 4809 1846 50  0000 L CNN
+F 1 "2K2" H 4809 1755 50  0000 L CNN
+F 2 "Resistor_SMD:R_0603_1608Metric" H 4750 1800 50  0001 C CNN
+F 3 "~" H 4750 1800 50  0001 C CNN
+	1    4750 1800
+	1    0    0    -1
+$EndComp
+$Comp
+L Device:D_Schottky D1
+U 1 1 60FAC885
+P 6600 2850
+F 0 "D1" V 6646 2770 50  0000 R CNN
+F 1 "B5819W" V 6555 2770 50  0000 R CNN
+F 2 "Diode_SMD:D_SOD-123" H 6600 2850 50  0001 C CNN
+F 3 "~" H 6600 2850 50  0001 C CNN
+	1    6600 2850
+	0    -1   -1   0
+$EndComp
+Wire Wire Line
+	6600 3100 6800 3100
+Connection ~ 6600 3100
+Wire Wire Line
+	7000 3100 7250 3100
+NoConn ~ 4200 4200
 $EndSCHEMATC

Commit message: Changed pull up resistor size for i2c to get basic part
Parts:
- C1: LCSC Part # (none) -> C19666
- C10, C11, C12: LCSC Part # (none) -> C13585
- C13, C14: LCSC Part # (none) -> C1547
- C2, C3, C4, C5, C6: LCSC Part # (none) -> C1525
- C7: LCSC Part # (none) -> C57112
- C8: LCSC Part # (none) -> C52923
- C9: LCSC Part # (none) -> C15195
- D1, D2: LCSC Part # (none) -> C8598
- D3: LCSC Part # (none) -> C72038
- D4: LCSC Part # (none) -> C72043
- F1: LCSC Part # (none) -> C369159
- FB1: LCSC Part # (none) -> C1017
- J4: footprint Connector_PinSocket_1.27mm:PinSocket_2x05_P1.27mm_Vertical_SMD -> Connector_PinHeader_1.27mm:PinHeader_2x05_P1.27mm_Vertical_SMD
- L1: LCSC Part # (none) -> C26443
- L2: LCSC Part # (none) -> C139506
Changed lines of the file:
@@
 F 2 "Capacitor_SMD:C_0402_1005Metric" H 1000 6100 50  0001 C CNN
 F 3 "~" H 1000 6100 50  0001 C CNN
+F 4 "C1547" H 1000 6100 50  0001 C CNN "LCSC Part #"
 	1    1000 6100
 	-1   0    0    1
@@
 F 2 "Capacitor_SMD:C_0402_1005Metric" H 1400 6100 50  0001 C CNN
 F 3 "~" H 1400 6100 50  0001 C CNN
+F 4 "C1547" H 1400 6100 50  0001 C CNN "LCSC Part #"
 	1    1400 6100
 	-1   0    0    1
@@
 F 2 "Inductor_SMD:L_0402_1005Metric" H 4400 2800 50  0001 C CNN
 F 3 "~" H 4400 2800 50  0001 C CNN
+F 4 "C26443" H 4400 2800 50  0001 C CNN "LCSC Part #"
 	1    4400 2800
 	0    -1   -1   0
@@
 F 2 "Capacitor_SMD:C_0402_1005Metric" H 4900 3100 50  0001 C CNN
 F 3 "~" H 4900 3100 50  0001 C CNN
+F 4 "C15195" H 4900 3100 50  0001 C CNN "LCSC Part #"
 	1    4900 3100
 	1    0    0    -1
@@
 F 2 "Capacitor_SMD:C_0402_1005Metric" H 4500 3100 50  0001 C CNN
 F 3 "~" H 4500 3100 50  0001 C CNN
+F 4 "C52923" H 4500 3100 50  0001 C CNN "LCSC Part #"
 	1    4500 3100
 	1    0    0    -1
@@
 F 2 "Capacitor_SMD:C_0603_1608Metric" H 1550 2800 50  0001 C CNN
 F 3 "~" H 1550 2800 50  0001 C CNN
+F 4 "C19666" H 1550 2800 50  0001 C CNN "LCSC Part #"
 	1    1550 2800
 	1    0    0    -1
@@
 F 2 "Capacitor_SMD:C_0402_1005Metric" H 2350 2800 50  0001 C CNN
 F 3 "~" H 2350 2800 50  0001 C CNN
+F 4 "C1525" H 2350 2800 50  0001 C CNN "LCSC Part #"
 	1    2350 2800
 	1    0    0    -1
@@
 F 2 "Capacitor_SMD:C_0402_1005Metric" H 2750 2800 50  0001 C CNN
 F 3 "~" H 2750 2800 50  0001 C CNN
+F 4 "C1525" H 2750 2800 50  0001 C CNN "LCSC Part #"
 	1    2750 2800
 	1    0    0    -1
@@
 F 2 "Capacitor_SMD:C_0402_1005Metric" H 3150 2800 50  0001 C CNN
 F 3 "~" H 3150 2800 50  0001 C CNN
+F 4 "C1525" H 3150 2800 50  0001 C CNN "LCSC Part #"
 	1    3150 2800
 	1    0    0    -1
@@
 F 2 "Capacitor_SMD:C_0402_1005Metric" H 1950 2800 50  0001 C CNN
 F 3 "~" H 1950 2800 50  0001 C CNN
+F 4 "C1525" H 1950 2800 50  0001 C CNN "LCSC Part #"
 	1    1950 2800
 	1    0    0    -1
@@
 F 2 "Capacitor_SMD:C_0402_1005Metric" H 3550 2800 50  0001 C CNN
 F 3 "~" H 3550 2800 50  0001 C CNN
+F 4 "C1525" H 3550 2800 50  0001 C CNN "LCSC Part #"
 	1    3550 2800
 	1    0    0    -1
@@
 F 0 "J4" H 1400 1617 50  0000 C CNN
 F 1 "SWD_Connector" H 1400 1526 50  0000 C CNN
-F 2 "Connector_PinSocket_1.27mm:PinSocket_2x05_P1.27mm_Vertical_SMD" H 1350 1200 50  0001 C CNN
+F 2 "Connector_PinHeader_1.27mm:PinHeader_2x05_P1.27mm_Vertical_SMD" H 1350 1200 50  0001 C CNN
 F 3 "~" H 1350 1200 50  0001 C CNN
 	1    1350 1200
@@
 F 2 "LED_SMD:LED_0603_1608Metric" V 2200 6800 50  0001 C CNN
 F 3 "~" V 2200 6800 50  0001 C CNN
+F 4 "C72043" H 2200 6800 50  0001 C CNN "LCSC Part #"
 	1    2200 6800
 	0    -1   -1   0
@@
 F 2 "LED_SMD:LED_0603_1608Metric" V 8450 5300 50  0001 C CNN
 F 3 "~" V 8450 5300 50  0001 C CNN
+F 4 "C72038" H 8450 5300 50  0001 C CNN "LCSC Part #"
 	1    8450 5300
 	0    -1   -1   0
@@
 F 2 "Fuse:Fuse_1206_3216Metric" H 6950 2900 50  0001 L CNN
 F 3 "~" H 6900 3100 50  0001 C CNN
+F 4 "C369159" H 6900 3100 50  0001 C CNN "LCSC Part #"
 	1    6900 3100
 	0    1    1    0
@@
 F 2 "Inductor_SMD:L_0805_2012Metric" V 7280 3100 50  0001 C CNN
 F 3 "~" H 7350 3100 50  0001 C CNN
+F 4 "C1017" H 7350 3100 50  0001 C CNN "LCSC Part #"
 	1    7350 3100
 	0    1    1    0
@@
 F 2 "Capacitor_SMD:C_0603_1608Metric" H 9900 2950 50  0001 C CNN
 F 3 "~" H 9900 2950 50  0001 C CNN
+F 4 "C57112" H 9900 2950 50  0001 C CNN "LCSC Part #"
 	1    9900 2950
 	0    1    1    0
@@
 F 2 "Diode_SMD:D_SOD-123" H 9950 3700 50  0001 C CNN
 F 3 "~" H 9950 3700 50  0001 C CNN
+F 4 "C8598" H 9950 3700 50  0001 C CNN "LCSC Part #"
 	1    9950 3700
 	0    1    1    0
@@
 F 2 "Inductor_SMD:L_Sunlord_MWSA0518_5.4x5.2mm" H 10250 3500 50  0001 C CNN
 F 3 "~" H 10250 3500 50  0001 C CNN
+F 4 "C139506" H 10250 3500 50  0001 C CNN "LCSC Part #"
 	1    10250 3500
 	0    -1   -1   0
@@
 F 2 "Capacitor_SMD:C_1206_3216Metric" H 7700 3300 50  0001 C CNN
 F 3 "~" H 7700 3300 50  0001 C CNN
+F 4 "C13585" H 7700 3300 50  0001 C CNN "LCSC Part #"
 	1    7700 3300
 	-1   0    0    1
@@
 F 2 "Capacitor_SMD:C_1206_3216Metric" H 10500 3650 50  0001 C CNN
 F 3 "~" H 10500 3650 50  0001 C CNN
+F 4 "C13585" H 10500 3650 50  0001 C CNN "LCSC Part #"
 	1    10500 3650
 	-1   0    0    1
@@
 F 2 "Capacitor_SMD:C_1206_3216Metric" H 10800 3650 50  0001 C CNN
 F 3 "~" H 10800 3650 50  0001 C CNN
+F 4 "C13585" H 10800 3650 50  0001 C CNN "LCSC Part #"
 	1    10800 3650
 	-1   0    0    1
@@
 F 2 "Diode_SMD:D_SOD-123" H 6600 2850 50  0001 C CNN
 F 3 "~" H 6600 2850 50  0001 C CNN
+F 4 "C8598" H 6600 2850 50  0001 C CNN "LCSC Part #"
 	1    6600 2850
 	0    -1   -1   0
