File: pcb/stm32l476rg_barebones/stm32l476rg.sch (KiCad schematic (older format))
At the start: 49 parts, among them J1 Conn_01x04_UART, J2 Conn_01x04_I2C, J3 Conn_01x06_SPI, J4 SWD_Connector, J5 USB_B_Micro, J6 Screw_Terminal_01x02, Q1 AO3401A, SW1 SW_SPDT, U1 USBLC6-2SC6, U2 MP2359DJ-LF-Z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

Commit message: Exported files for manufacturing
Parts:
- Y1: LCSC Part # (none) -> C13738
Changed lines of the file:
@@
 F 2 "Crystal:Crystal_SMD_3225-4Pin_3.2x2.5mm" H 1200 5600 50  0001 C CNN
 F 3 "~" H 1200 5600 50  0001 C CNN
+F 4 "C13738" H 1200 5600 50  0001 C CNN "LCSC Part #"
 	1    1200 5600
 	1    0    0    -1
